File: Platinen/Motorsteuerung/motorsteuerung.kicad_pcb (KiCad board)
At the start: 2 copper layers, 13 parts, among them J1 CONN_01X08, J2 CONN_01X08, J3 CONN_01X02, J4 CONN_01X04, J5 CONN_01X02, J6 CONN_01X02, J7 CONN_01X01, P2 CONN_01X04, U1 L293D

Commit message: Platinen aktuallisiert nach Ätzen der ersten Prototypplatine
Parts:
- added R5: 0, Resistors_THT:R_Axial_DIN0204_L3.6mm_D1.6mm_P7.62mm_Horizontal, F.Cu at (64.8, 54.6)
- R2: footprint Resistors_THT:R_Axial_DIN0207_L6.3mm_D2.5mm_P15.24mm_Horizontal -> Resistors_THT:R_Axial_DIN0309_L9.0mm_D3.2mm_P20.32mm_Horizontal
- moved R1 35.1 mm to (64.8, 57.1), turned to 0 degrees
- moved J2 21.0 mm to (74.9, 64.8)
- moved J3 18.5 mm to (35.6, 53.3)
- moved P2 8.89 mm to (34.3, 59.7)
- moved J5 6.35 mm to (45.7, 59.7)
- moved J6 6.35 mm to (49.5, 59.7)
- moved R2 1.27 mm to (40.6, 30.5)
Connections:
- J2 pad 1: Net-(J2-Pad1) -> Net-(J1-Pad8)
- J2 pad 5: Net-(J2-Pad1) -> Net-(J1-Pad8)
- J2 pad 8: Net-(J1-Pad8) -> Net-(J2-Pad4)
- J3 pad 1: Net-(J1-Pad8) -> Net-(J3-Pad1)
- J3 pad 2: Net-(J2-Pad1) -> Net-(J1-Pad8)
- J5 pad 1: Net-(J1-Pad8) -> Net-(J3-Pad1)
- J5 pad 2: Net-(J2-Pad1) -> Net-(J1-Pad8)
- J6 pad 1: Net-(J1-Pad8) -> Net-(J3-Pad1)
- J6 pad 2: Net-(J2-Pad1) -> Net-(J1-Pad8)
- P2 pad 1: Net-(J1-Pad8) -> Net-(J3-Pad1)
- P2 pad 4: Net-(J2-Pad1) -> Net-(J1-Pad8)
- R1 pad 1: Net-(J1-Pad8) -> Net-(J3-Pad1)
- R2 pad 2: Net-(J2-Pad1) -> Net-(J3-Pad1)
Routing:
- net Net-(J1-Pad8): track 123.0 -> 0.00 mm
- net Net-(J2-Pad1): track 103.9 -> 0.00 mm
- net Net-(J3-Pad1): track 0.00 -> 47.3 mm
- net Net-(J2-Pad7): track 25.7 -> 55.4 mm
- net Net-(J2-Pad3): track 37.4 -> 67.1 mm
- net Net-(J2-Pad6): track 33.2 -> 62.2 mm
- net Net-(J2-Pad2): track 24.7 -> 45.9 mm
- net Net-(J2-Pad4): track 3.81 -> 16.3 mm
