File: Platinen/Motorsteuerung/motorsteuerung.sch (KiCad schematic (older format))
At the start: 13 parts, among them J1 CONN_01X08, J2 CONN_01X08, J3 CONN_01X02, J4 CONN_01X04, J5 CONN_01X02, J6 CONN_01X02, J7 CONN_01X01, P2 CONN_01X04, U1 L293D

Commit message: Platinen aktuallisiert nach Ätzen der ersten Prototypplatine
Parts:
- added R5: 0, Resistors_THT:R_Axial_DIN0204_L3.6mm_D1.6mm_P7.62mm_Horizontal, symbol R
- J1, J2: symbol CONN_01X08 -> Conn_01x08
- J3, J5, J6: symbol CONN_01X02 -> Conn_01x02
- J4, P2: symbol CONN_01X04 -> Conn_01x04
- J7: symbol CONN_01X01 -> Conn_01x01
- R2: footprint Resistors_THT:R_Axial_DIN0207_L6.3mm_D2.5mm_P15.24mm_Horizontal -> Resistors_THT:R_Axial_DIN0309_L9.0mm_D3.2mm_P20.32mm_Horizontal
Connections:
- wire segments 71 -> 73
Other:
- moved on the sheet: R1
