File: Platinen/RGB/rgb.sch (KiCad schematic (older format))
At the start: 5 parts, among them J1 CONN_01X04_FEMALE

Commit message: Platinen aktuallisiert nach Ätzen der ersten Prototypplatine
Parts:
- J1: symbol CONN_01X04_FEMALE -> Conn_01x04_Female
Connections:
- wire segments 8 -> 13
Changed lines of the file:
@@
 EESchema Schematic File Version 2
+LIBS:rgb-rescue
 LIBS:power
 LIBS:device
@@
 LIBS:contrib
 LIBS:valves
-LIBS:rgb-cache
 EELAYER 25 0
 EELAYER END
@@
 $EndDescr
 $Comp
-L CONN_01X04_FEMALE J1
+L Conn_01x04_Female J1
 U 1 1 58B815B1
-P 5100 2250
-F 0 "J1" H 5100 2650 50  0000 C CNN
-F 1 "CONN_01X04_FEMALE" H 5200 1850 50  0000 C CNN
-F 2 "Pin_Headers:Pin_Header_Straight_1x04_Pitch2.54mm" H 5100 2550 50  0001 C CNN
-F 3 "" H 5100 2550 50  0001 C CNN
-	1    5100 2250
+P 5300 2150
+F 0 "J1" H 5300 2550 50  0000 C CNN
+F 1 "CONN_01X04_FEMALE" H 5400 1750 50  0000 C CNN
+F 2 "Pin_Headers:Pin_Header_Straight_1x04_Pitch2.54mm" H 5300 2450 50  0001 C CNN
+F 3 "" H 5300 2450 50  0001 C CNN
+	1    5300 2150
 	1    0    0    -1
 $EndComp
@@
 	5000 1950 4500 1950
 Wire Wire Line
-	4500 2150 5000 2150
+	4500 2150 5100 2150
 Wire Wire Line
 	5000 2350 4500 2350
@@
 	3450 2150 3450 2550
 Wire Wire Line
-	3450 2550 5000 2550
+	3450 2550 5100 2550
+Wire Wire Line
+	5000 1950 5000 2050
+Wire Wire Line
+	5000 2050 5100 2050
+Wire Wire Line
+	5100 2250 5000 2250
+Wire Wire Line
+	5000 2250 5000 2350
+Wire Wire Line
+	5100 2550 5100 2350
 $EndSCHEMATC
