File: Platinen/RGB/rgb.kicad_pcb (KiCad board)
At the start: 2 copper layers, 5 parts, among them J1 CONN_01X04_FEMALE

Commit message: Platinen aktuallisiert nach Ätzen der ersten Prototypplatine
Routing:
- net Net-(D1-Pad1): track 34.5 -> 0.00 mm
Changed lines of the file:
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@@
-(kicad_pcb (version 4) (host pcbnew 4.0.6-e0-6349~53~ubuntu14.04.1)
+(kicad_pcb (version 4) (host pcbnew 4.0.7-e2-6376~58~ubuntu16.04.1)
   (general
     (links 7)
     (no_connects 0)
-    (area 0 0 0 0)
+    (area 17.78 17.78 54.610001 33.020001)
     (thickness 1.6)
-    (drawings 0)
-    (tracks 22)
+    (drawings 1)
+    (tracks 17)
     (zones 0)
     (modules 5)
@@
     )
   )
-  (segment (start 22.86 25.654) (end 21.336 25.654) (width 0.5) (layer B.Cu) (net 1))
-  (segment (start 20.32 31.75) (end 43.18 31.75) (width 0.5) (layer B.Cu) (net 1))
-  (segment (start 43.18 31.75) (end 45.72 29.21) (width 0.5) (layer B.Cu) (net 1))
-  (segment (start 20.32 26.67) (end 20.32 31.75) (width 0.5) (layer B.Cu) (net 1))
-  (segment (start 21.336 25.654) (end 20.32 26.67) (width 0.5) (layer B.Cu) (net 1))
+  (dimension 10.16 (width 0.3) (layer F.Adhes)
+    (gr_text "10,160 mm" (at 52.07 15.16) (layer F.Adhes)
+      (effects (font (size 1.5 1.5) (thickness 0.3)))
+    )
+    (feature1 (pts (xy 57.15 17.78) (xy 57.15 13.81)))
+    (feature2 (pts (xy 46.99 17.78) (xy 46.99 13.81)))
+    (crossbar (pts (xy 46.99 16.51) (xy 57.15 16.51)))
+    (arrow1a (pts (xy 57.15 16.51) (xy 56.023496 17.096421)))
+    (arrow1b (pts (xy 57.15 16.51) (xy 56.023496 15.923579)))
+    (arrow2a (pts (xy 46.99 16.51) (xy 48.116504 17.096421)))
+    (arrow2b (pts (xy 46.99 16.51) (xy 48.116504 15.923579)))
+  )
   (segment (start 30.48 21.59) (end 25.4 21.59) (width 0.5) (layer B.Cu) (net 2))
   (segment (start 21.082 23.622) (end 22.86 23.622) (width 0.5) (layer B.Cu) (net 2))
@@
   (segment (start 24.13 21.59) (end 25.4 22.86) (width 0.5) (layer B.Cu) (net 3))
   (segment (start 25.4 22.86) (end 29.21 22.86) (width 0.5) (layer B.Cu) (net 3))
-  (segment (start 29.21 22.86) (end 30.48 24.13) (width 0.5) (layer B.Cu) (net 3))
+  (segment (start 29.21 22.86) (end 30.48 24.13) (width 0.5) (layer B.Cu) (net 3) (status 20))
   (segment (start 30.48 26.67) (end 26.67 26.67) (width 0.5) (layer B.Cu) (net 4))
   (segment (start 25.654 27.686) (end 22.86 27.686) (width 0.5) (layer B.Cu) (net 4))
   (segment (start 26.67 26.67) (end 25.654 27.686) (width 0.5) (layer B.Cu) (net 4))
-  (segment (start 45.72 24.13) (end 40.64 24.13) (width 0.5) (layer B.Cu) (net 5))
+  (segment (start 45.72 24.13) (end 40.64 24.13) (width 0.5) (layer B.Cu) (net 5) (status 20))
   (segment (start 40.64 21.59) (end 45.72 21.59) (width 0.5) (layer B.Cu) (net 6))
   (segment (start 40.64 26.67) (end 45.72 26.67) (width 0.5) (layer B.Cu) (net 7))
@@
     (polygon
       (pts
-        (xy 54.61 33.02) (xy 17.78 33.02) (xy 17.78 17.78) (xy 54.61 17.78)
+        (xy 57.15 33.02) (xy 17.78 33.02) (xy 17.78 17.78) (xy 57.15 17.78)
       )
     )

Commit message: Platinen überarbeitet
Parts:
- moved J1 2.54 mm to (43.2, 21.6)
- moved R1 1.27 mm to (39.4, 21.6)
- moved R2 1.27 mm to (39.4, 24.1)
- moved R3 1.27 mm to (39.4, 26.7)
Routing:
- net Net-(D1-Pad4): track 8.04 -> 6.77 mm
- net Net-(J1-Pad3): track 5.08 -> 3.81 mm
- net Net-(J1-Pad2): track 5.08 -> 3.81 mm
- net Net-(J1-Pad1): track 5.08 -> 3.81 mm
Other:
- net class Default: trace_width 0.5 -> 0.75
- board text added: "Blau"
- board text added: "GND"
- board text added: "Grün"
- board text added: "Rot"
Changed lines of the file:
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@@
     (links 7)
     (no_connects 0)
-    (area 17.78 17.78 54.610001 33.020001)
+    (area 17.925 13.81 58.57 32.675)
     (thickness 1.6)
-    (drawings 1)
+    (drawings 5)
     (tracks 17)
     (zones 0)
@@
   )
   (setup
-    (last_trace_width 0.5)
+    (last_trace_width 0.75)
     (trace_clearance 0.2)
-    (zone_clearance 0.508)
+    (zone_clearance 0.8)
     (zone_45_only no)
     (trace_min 0.2)
@@
     (pad_drill 0.8)
     (pad_to_mask_clearance 0.2)
-    (aux_axis_origin 0 0)
+    (aux_axis_origin 19.05 31.75)
+    (grid_origin 19.05 31.75)
     (visible_elements FFFFFF7F)
     (pcbplotparams
-      (layerselection 0x00030_80000001)
+      (layerselection 0x00008_80000000)
       (usegerberextensions false)
       (excludeedgelayer true)
@@
       (viasonmask false)
       (mode 1)
-      (useauxorigin false)
+      (useauxorigin true)
       (hpglpennumber 1)
       (hpglpenspeed 20)
@@
       (psnegative false)
       (psa4output false)
-      (plotreference true)
-      (plotvalue true)
+      (plotreference false)
+      (plotvalue false)
       (plotinvisibletext false)
       (padsonsilk false)
@@
       (outputformat 1)
       (mirror false)
-      (drillshape 1)
+      (drillshape 0)
       (scaleselection 1)
       (outputdirectory ""))
@@
   (net_class Default "Dies ist die voreingestellte Netzklasse."
     (clearance 0.2)
-    (trace_width 0.5)
+    (trace_width 0.75)
     (via_dia 0.6)
     (via_drill 0.4)
@@
   )
   (module Resistors_THT:R_Axial_DIN0207_L6.3mm_D2.5mm_P10.16mm_Horizontal (layer F.Cu)
-    (at 40.64 24.13 180)
+    (at 39.37 24.13 180)
     (descr "Resistor, Axial_DIN0207 series, Axial, Horizontal, pin pitch=10.16mm, 0.25W = 1/4W, length*diameter=6.3*2.5mm^2, http://cdn-reichelt.de/documents/datenblatt/B400/1_4W%23YAG.pdf")
     (tags "Resistor Axial_DIN0207 series Axial Horizontal pin pitch 10.16mm 0.25W = 1/4W length 6.3mm diameter 2.5mm")
@@
   )
   (module Pin_Headers:Pin_Header_Straight_1x04_Pitch2.54mm (layer F.Cu)
-    (at 45.72 21.59)
+    (at 43.18 21.59)
     (descr "Through hole straight pin header, 1x04, 2.54mm pitch, single row")
     (tags "Through hole pin header THT 1x04 2.54mm single row")
@@
   )
   (module Resistors_THT:R_Axial_DIN0207_L6.3mm_D2.5mm_P10.16mm_Horizontal (layer F.Cu)
-    (at 40.64 21.59 180)
+    (at 39.37 21.59 180)
     (descr "Resistor, Axial_DIN0207 series, Axial, Horizontal, pin pitch=10.16mm, 0.25W = 1/4W, length*diameter=6.3*2.5mm^2, http://cdn-reichelt.de/documents/datenblatt/B400/1_4W%23YAG.pdf")
     (tags "Resistor Axial_DIN0207 series Axial Horizontal pin pitch 10.16mm 0.25W = 1/4W length 6.3mm diameter 2.5mm")
@@
   )
   (module Resistors_THT:R_Axial_DIN0207_L6.3mm_D2.5mm_P10.16mm_Horizontal (layer F.Cu)
-    (at 40.64 26.67 180)
+    (at 39.37 26.67 180)
     (descr "Resistor, Axial_DIN0207 series, Axial, Horizontal, pin pitch=10.16mm, 0.25W = 1/4W, length*diameter=6.3*2.5mm^2, http://cdn-reichelt.de/documents/datenblatt/B400/1_4W%23YAG.pdf")
     (tags "Resistor Axial_DIN0207 series Axial Horizontal pin pitch 10.16mm 0.25W = 1/4W length 6.3mm diameter 2.5mm")
@@
     )
   )
+  (gr_text GND (at 45.72 29.21) (layer F.Paste)
+    (effects (font (size 1.8 1.8) (thickness 0.1)) (justify left))
+  )
+  (gr_text Blau (at 45.72 26.67) (layer F.Paste)
+    (effects (font (size 1.8 1.8) (thickness 0.1)) (justify left))
+  )
+  (gr_text Grün (at 45.72 24.13) (layer F.Paste)
+    (effects (font (size 1.8 1.8) (thickness 0.1)) (justify left))
+  )
+  (gr_text Rot (at 45.72 21.59) (layer F.Paste)
+    (effects (font (size 1.8 1.8) (thickness 0.1)) (justify left))
+  )
   (dimension 10.16 (width 0.3) (layer F.Adhes)
     (gr_text "10,160 mm" (at 52.07 15.16) (layer F.Adhes)
@@
     (arrow2b (pts (xy 46.99 16.51) (xy 48.116504 15.923579)))
   )
-  (segment (start 30.48 21.59) (end 25.4 21.59) (width 0.5) (layer B.Cu) (net 2))
-  (segment (start 21.082 23.622) (end 22.86 23.622) (width 0.5) (layer B.Cu) (net 2))
-  (segment (start 20.32 22.86) (end 21.082 23.622) (width 0.5) (layer B.Cu) (net 2))
-  (segment (start 20.32 21.59) (end 20.32 22.86) (width 0.5) (layer B.Cu) (net 2))
-  (segment (start 21.59 20.32) (end 20.32 21.59) (width 0.5) (layer B.Cu) (net 2))
-  (segment (start 24.13 20.32) (end 21.59 20.32) (width 0.5) (layer B.Cu) (net 2))
-  (segment (start 25.4 21.59) (end 24.13 20.32) (width 0.5) (layer B.Cu) (net 2))
-  (segment (start 22.86 21.59) (end 24.13 21.59) (width 0.5) (layer B.Cu) (net 3))
-  (segment (start 24.13 21.59) (end 25.4 22.86) (width 0.5) (layer B.Cu) (net 3))
-  (segment (start 25.4 22.86) (end 29.21 22.86) (width 0.5) (layer B.Cu) (net 3))
-  (segment (start 29.21 22.86) (end 30.48 24.13) (width 0.5) (layer B.Cu) (net 3) (status 20))
-  (segment (start 30.48 26.67) (end 26.67 26.67) (width 0.5) (layer B.Cu) (net 4))
-  (segment (start 25.654 27.686) (end 22.86 27.686) (width 0.5) (layer B.Cu) (net 4))
-  (segment (start 26.67 26.67) (end 25.654 27.686) (width 0.5) (layer B.Cu) (net 4))
-  (segment (start 45.72 24.13) (end 40.64 24.13) (width 0.5) (layer B.Cu) (net 5) (status 20))
-  (segment (start 40.64 21.59) (end 45.72 21.59) (width 0.5) (layer B.Cu) (net 6))
-  (segment (start 40.64 26.67) (end 45.72 26.67) (width 0.5) (layer B.Cu) (net 7))
+  (segment (start 22.86 23.622) (end 21.082 23.622) (width 0.75) (layer B.Cu) (net 2))
+  (segment (start 26.035 21.59) (end 29.21 21.59) (width 0.75) (layer B.Cu) (net 2))
+  (segment (start 24.13 19.685) (end 26.035 21.59) (width 0.75) (layer B.Cu) (net 2))
+  (segment (start 21.59 19.685) (end 24.13 19.685) (width 0.75) (layer B.Cu) (net 2))
+  (segment (start 20.32 20.955) (end 21.59 19.685) (width 0.75) (layer B.Cu) (net 2))
+  (segment (start 20.32 22.86) (end 20.32 20.955) (width 0.75) (layer B.Cu) (net 2))
+  (segment (start 21.082 23.622) (end 20.32 22.86) (width 0.75) (layer B.Cu) (net 2))
+  (segment (start 22.86 21.59) (end 24.056494 21.59) (width 0.75) (layer B.Cu) (net 3) (status 400030))
+  (segment (start 24.056494 21.59) (end 26.596494 24.13) (width 0.75) (layer B.Cu) (net 3) (status 10))
+  (segment (start 26.596494 24.13) (end 29.21 24.13) (width 0.75) (layer B.Cu) (net 3) (status 800000))
+  (segment (start 22.86 21.59) (end 24.13 21.59) (width 0.5) (layer B.Cu) (net 3) (status 400030))
+  (segment (start 29.21 26.67) (end 25.4 26.67) (width 0.75) (layer B.Cu) (net 4))
+  (segment (start 24.384 27.686) (end 22.86 27.686) (width 0.75) (layer B.Cu) (net 4) (status 20))
+  (segment (start 25.4 26.67) (end 24.384 27.686) (width 0.75) (layer B.Cu) (net 4))
+  (segment (start 43.18 24.13) (end 39.37 24.13) (width 0.75) (layer B.Cu) (net 5) (status 10))
+  (segment (start 39.37 21.59) (end 43.18 21.59) (width 0.75) (layer B.Cu) (net 6) (status 20))
+  (segment (start 39.37 26.67) (end 43.18 26.67) (width 0.75) (layer B.Cu) (net 7) (status 20))
   (zone (net 1) (net_name "Net-(D1-Pad1)") (layer B.Cu) (hatch edge 0.508)
-    (connect_pads (clearance 0.508))
-    (min_thickness 0.254)
-    (fill yes (arc_segments 16) (thermal_gap 0.508) (thermal_bridge_width 0.508))
+    (connect_pads (clearance 0.8))
+    (min_thickness 0.7)
+    (fill yes (arc_segments 16) (thermal_gap 0.8) (thermal_bridge_width 0.8))
     (polygon
       (pts
-        (xy 57.15 33.02) (xy 17.78 33.02) (xy 17.78 17.78) (xy 57.15 17.78)
+        (xy 53.34 31.75) (xy 19.05 31.75) (xy 19.05 19.05) (xy 53.34 19.05)
       )
     )
