File: Platinen/AD-Wandler/adwandler.sch (KiCad schematic (older format))
At the start: 6 parts, among them J1 CONN_01X06, U1 MCP3208

Commit message: Platinen aktuallisiert nach Ätzen der ersten Prototypplatine
Parts:
- J1: symbol CONN_01X06 -> Conn_01x06
Changed lines of the file:
@@
 EESchema Schematic File Version 2
+LIBS:adwandler-rescue
 LIBS:power
 LIBS:device
@@
 $EndComp
 $Comp
-L CONN_01X06 J1
+L Conn_01x06 J1
 U 1 1 58B30941
-P 8100 3950
-F 0 "J1" H 8100 4300 50  0000 C CNN
-F 1 "CONN_01X06" V 8200 3950 50  0000 C CNN
-F 2 "adwandler:Socket_Strip_Straight_1x06_Pitch2.54mm_breit" H 8100 3950 50  0001 C CNN
-F 3 "" H 8100 3950 50  0001 C CNN
-	1    8100 3950
+P 8100 3900
+F 0 "J1" H 8100 4250 50  0000 C CNN
+F 1 "CONN_01X06" V 8200 3900 50  0000 C CNN
+F 2 "adwandler:Socket_Strip_Straight_1x06_Pitch2.54mm_breit" H 8100 3900 50  0001 C CNN
+F 3 "" H 8100 3900 50  0001 C CNN
+	1    8100 3900
 	1    0    0    -1
 $EndComp

Commit message: Schaltpläne überarbeitet
Parts:
- J1: symbol Conn_01x06 -> adwandler-rescue:Conn_01x06
- RV1, RV2, RV3, RV4: symbol POT -> adwandler-rescue:POT
- U1: symbol MCP3208 -> adwandler-rescue:MCP3208
Changed lines of the file:
@@
-EESchema Schematic File Version 2
-LIBS:adwandler-rescue
-LIBS:power
-LIBS:device
-LIBS:transistors
-LIBS:conn
-LIBS:linear
-LIBS:regul
-LIBS:74xx
-LIBS:cmos4000
-LIBS:adc-dac
-LIBS:memory
-LIBS:xilinx
-LIBS:microcontrollers
-LIBS:dsp
-LIBS:microchip
-LIBS:analog_switches
-LIBS:motorola
-LIBS:texas
-LIBS:intel
-LIBS:audio
-LIBS:interface
-LIBS:digital-audio
-LIBS:philips
-LIBS:display
-LIBS:cypress
-LIBS:siliconi
-LIBS:opto
-LIBS:atmel
-LIBS:contrib
-LIBS:valves
+EESchema Schematic File Version 4
 LIBS:adwandler-cache
-EELAYER 25 0
+EELAYER 26 0
 EELAYER END
 $Descr A4 11693 8268
@@
 $EndDescr
 $Comp
-L POT RV1
+L adwandler-rescue:POT RV1
 U 1 1 58B30835
 P 4700 3300
@@
 $EndComp
 $Comp
-L POT RV2
+L adwandler-rescue:POT RV2
 U 1 1 58B30844
 P 4700 3700
@@
 $EndComp
 $Comp
-L POT RV3
+L adwandler-rescue:POT RV3
 U 1 1 58B30853
 P 4700 4100
@@
 $EndComp
 $Comp
-L POT RV4
+L adwandler-rescue:POT RV4
 U 1 1 58B30862
 P 4650 4650
@@
 $EndComp
 $Comp
-L Conn_01x06 J1
+L adwandler-rescue:Conn_01x06 J1
 U 1 1 58B30941
 P 8100 3900
@@
 $EndComp
 Wire Wire Line
-	6250 4200 7900 4200
+	6250 4200 7400 4200
 Wire Wire Line
-	5950 4100 5950 5050
-Connection ~ 7400 4100
+	5950 4100 5950 4400
 Wire Wire Line
-	6250 3000 7250 3000
+	6250 3000 6500 3000
 Wire Wire Line
 	7250 3000 7250 4100
@@
 	5950 3000 5950 2800
 Wire Wire Line
-	4700 2800 6500 2800
+	4700 2800 5950 2800
 Wire Wire Line
 	6500 2800 6500 3000
 Connection ~ 6500 3000
-Wire Wire Line
-	7250 4100 7900 4100
 Wire Wire Line
 	6650 3700 7900 3700
@@
 	4700 3150 4250 3150
 Wire Wire Line
-	4250 3150 4250 4500
+	4250 3150 4250 3550
 Wire Wire Line
 	4250 4500 4650 4500
@@
 	4650 4800 5200 4800
 Wire Wire Line
-	5200 4800 5200 3450
+	5200 4800 5200 4250
 Wire Wire Line
 	5200 3450 4700 3450
@@
 	4850 3200 4850 3300
 $Comp
-L MCP3208 U1
+L adwandler-rescue:MCP3208 U1
 U 1 1 58B34079
 P 6050 3500
@@
 	7400 4400 5950 4400
 Connection ~ 7400 4200
+Wire Wire Line
+	6500 3000 7250 3000
+Wire Wire Line
+	5950 2800 6500 2800
+Wire Wire Line
+	4250 3950 4250 4500
+Wire Wire Line
+	4250 3550 4250 3950
+Wire Wire Line
+	5950 4400 5950 5050
+Wire Wire Line
+	5200 3850 5200 3450
+Wire Wire Line
+	5200 4250 5200 3850
+Wire Wire Line
+	7400 4200 7900 4200
+Wire Wire Line
+	7250 4100 7900 4100
 $EndSCHEMATC
