File: Platinen/AD-Wandler/adwandler.kicad_pcb (KiCad board)
At the start: 2 copper layers, 6 parts, among them J1 CONN_01X06, U1 MCP3208

Commit message: Platinen aktuallisiert nach Ätzen der ersten Prototypplatine
Parts:
- moved RV4 5.08 mm to (22.9, 64.8)
- moved RV1 2.54 mm to (22.9, 30.5)
- moved RV3 2.54 mm to (22.9, 53.3)
Routing:
- net Net-(J1-Pad6): track 153.6 -> 0.11 mm
- net Net-(J1-Pad5): track 107.9 -> 95.2 mm
- net Net-(RV4-Pad2): track 26.6 -> 21.6 mm
- net Net-(RV3-Pad2): track 15.2 -> 12.8 mm
- net Net-(RV1-Pad2): track 15.1 -> 12.8 mm

Commit message: Schaltpläne überarbeitet
Parts:
- moved J1 10.2 mm to (48.3, 51.4)
- moved U1 5.12 mm to (36.8, 36.2)
Routing:
- net Net-(J1-Pad5): track 95.2 -> 83.8 mm
- net Net-(J1-Pad4): track 9.52 -> 3.81 mm
- net Net-(J1-Pad3): track 9.52 -> 3.81 mm
- net Net-(J1-Pad2): track 9.52 -> 3.81 mm
- net Net-(J1-Pad1): track 9.52 -> 3.81 mm
- net Net-(RV2-Pad2): track 9.12 -> 5.32 mm
- net Net-(RV1-Pad2): track 12.8 -> 9.86 mm
- net Net-(J1-Pad6): track 0.11 -> 1.38 mm
- net Net-(RV4-Pad2): track 21.6 -> 22.7 mm
- net Net-(RV3-Pad2): track 12.8 -> 12.0 mm
Other:
- net class Breite: trace_width 0.5 -> 0.75
- net class Default: trace_width 0.5 -> 0.75
- board text added: "3,3V"
- board text added: "GND"
- board text added: "IO10"
- board text added: "IO11"
- board text added: "IO8"
- board text added: "IO9"
Changed lines of the file:
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@@
-(kicad_pcb (version 4) (host pcbnew 4.0.7-e2-6376~58~ubuntu16.04.1)
+(kicad_pcb (version 4) (host pcbnew 4.0.7-e2-6376~58~ubuntu14.04.1)
   (general
     (links 20)
     (no_connects 0)
-    (area 19.685 10 72.54 74.930001)
+    (area 19.685 10 72.54 69.495)
     (thickness 1.6)
-    (drawings 1)
-    (tracks 30)
+    (drawings 7)
+    (tracks 40)
     (zones 0)
     (modules 6)
@@
   )
   (setup
-    (last_trace_width 0.5)
+    (last_trace_width 0.75)
     (trace_clearance 0.2)
-    (zone_clearance 0.508)
+    (zone_clearance 0.8)
     (zone_45_only no)
     (trace_min 0.2)
@@
     (visible_elements FFFFFF7F)
     (pcbplotparams
-      (layerselection 0x00030_80000001)
+      (layerselection 0x00008_80000000)
       (usegerberextensions false)
       (excludeedgelayer true)
@@
       (outputformat 1)
       (mirror false)
-      (drillshape 1)
+      (drillshape 0)
       (scaleselection 1)
       (outputdirectory ""))
@@
   (net_class Default "Dies ist die voreingestellte Netzklasse."
     (clearance 0.2)
-    (trace_width 0.5)
+    (trace_width 0.75)
     (via_dia 0.6)
     (via_drill 0.4)
@@
   (net_class Breite ""
     (clearance 0.2)
-    (trace_width 0.5)
+    (trace_width 0.75)
     (via_dia 0.6)
     (via_drill 0.4)
@@
   )
   (module adwandler:DIP-16_W7.62mm_bigpads (layer F.Cu)
-    (at 41.91 36.83)
+    (at 36.83 36.195)
     (descr "16-lead dip package, row spacing 7.62 mm (300 mils)")
     (tags "DIL DIP PDIP 2.54mm 7.62mm 300mil")
@@
   )
   (module adwandler:Socket_Strip_Straight_1x06_Pitch2.54mm_breit (layer F.Cu)
-    (at 58.42 52.07 180)
+    (at 48.26 51.435 180)
     (descr "Through hole straight socket strip, 1x06, 2.54mm pitch, single row")
     (tags "Through hole socket strip THT 1x06 2.54mm single row")
@@
     )
   )
+  (gr_text IO8 (at 50.165 51.435) (layer F.Paste)
+    (effects (font (size 1.8 1.8) (thickness 0.1)) (justify left))
+  )
+  (gr_text IO10 (at 50.165 48.895) (layer F.Paste)
+    (effects (font (size 1.8 1.8) (thickness 0.1)) (justify left))
+  )
+  (gr_text IO9 (at 50.165 46.355) (layer F.Paste)
+    (effects (font (size 1.8 1.8) (thickness 0.1)) (justify left))
+  )
+  (gr_text IO11 (at 50.165 43.815) (layer F.Paste)
+    (effects (font (size 1.8 1.8) (thickness 0.1)) (justify left))
+  )
+  (gr_text 3,3V (at 50.165 41.275) (layer F.Paste)
+    (effects (font (size 1.8 1.8) (thickness 0.1)) (justify left))
+  )
+  (gr_text GND (at 50.165 38.735) (layer F.Paste)
+    (effects (font (size 1.8 1.8) (thickness 0.1)) (justify left))
+  )
   (dimension 10.16 (width 0.3) (layer F.Adhes)
     (gr_text "10,160 mm" (at 66.04 11.35) (layer F.Adhes)
@@
   )
   (segment (start 22.86 50.88) (end 22.94 50.8) (width 0.25) (layer F.Cu) (net 0))
-  (segment (start 41.91 36.83) (end 32.86 27.78) (width 0.5) (layer B.Cu) (net 1))
-  (segment (start 49.53 52.07) (end 59.055 52.07) (width 0.5) (layer B.Cu) (net 2))
-  (segment (start 41.91 39.37) (end 32.9 39.37) (width 0.5) (layer B.Cu) (net 3))
+  (segment (start 36.83 36.195) (end 36.83 31.95) (width 0.75) (layer B.Cu) (net 1))
+  (segment (start 36.83 31.95) (end 32.86 27.98) (width 0.75) (layer B.Cu) (net 1))
+  (segment (start 44.45 51.435) (end 48.26 51.435) (width 0.75) (layer B.Cu) (net 2))
+  (segment (start 36.83 38.735) (end 33.535 38.735) (width 0.75) (layer B.Cu) (net 3))
+  (segment (start 33.535 38.735) (end 32.86 39.41) (width 0.75) (layer B.Cu) (net 3))
+  (segment (start 33.535 38.735) (end 32.86 39.41) (width 0.75) (layer B.Cu) (net 3))
   (segment (start 32.9 39.37) (end 32.86 39.41) (width 0.25) (layer B.Cu) (net 3))
-  (segment (start 41.91 39.37) (end 41.87 39.41) (width 0.25) (layer F.Cu) (net 3))
-  (segment (start 59.055 49.53) (end 49.53 49.53) (width 0.5) (layer B.Cu) (net 4))
-  (segment (start 41.91 41.91) (end 32.86 50.96) (width 0.5) (layer B.Cu) (net 5))
-  (segment (start 59.055 46.99) (end 49.53 46.99) (width 0.5) (layer B.Cu) (net 6))
+  (segment (start 36.83 38.735) (end 36.79 38.775) (width 0.25) (layer F.Cu) (net 3) (status 30))
+  (segment (start 44.45 48.895) (end 48.26 48.895) (width 0.75) (layer B.Cu) (net 4))
+  (segment (start 36.83 41.275) (end 35.56 41.275) (width 0.75) (layer B.Cu) (net 5))
+  (segment (start 35.56 41.275) (end 32.86 43.975) (width 0.75) (layer B.Cu) (net 5))
+  (segment (start 32.86 43.975) (end 32.86 50.84) (width 0.75) (layer B.Cu) (net 5))
+  (segment (start 48.26 46.355) (end 44.45 46.355) (width 0.75) (layer B.Cu) (net 6))
+  (segment (start 36.83 43.815) (end 37.465 43.815) (width 0.75) (layer B.Cu) (net 7))
+  (segment (start 37.465 43.815) (end 39.37 45.72) (width 0.75) (layer B.Cu) (net 7))
+  (segment (start 39.37 45.72) (end 39.37 55.76) (width 0.75) (layer B.Cu) (net 7))
+  (segment (start 39.37 55.76) (end 32.86 62.27) (width 0.75) (layer B.Cu) (net 7))
   (segment (start 32.86 62.27) (end 32.98 62.27) (width 0.5) (layer B.Cu) (net 7))
-  (segment (start 32.98 62.27) (end 35.56 59.69) (width 0.5) (layer B.Cu) (net 7))
-  (segment (start 35.56 59.69) (end 35.56 50.8) (width 0.5) (layer B.Cu) (net 7))
-  (segment (start 35.56 50.8) (end 41.91 44.45) (width 0.5) (layer B.Cu) (net 7))
-  (segment (start 49.53 44.45) (end 59.055 44.45) (width 0.5) (layer B.Cu) (net 8))
-  (segment (start 25.4 53.34) (end 25.4 62.23) (width 0.5) (layer B.Cu) (net 10))
-  (segment (start 25.4 62.23) (end 22.86 64.77) (width 0.5) (layer B.Cu) (net 10))
-  (segment (start 25.4 41.91) (end 25.4 53.34) (width 0.5) (layer B.Cu) (net 10))
-  (segment (start 25.4 53.34) (end 22.86 53.34) (width 0.5) (layer B.Cu) (net 10))
-  (segment (start 49.53 39.37) (end 52.07 41.91) (width 0.5) (layer B.Cu) (net 10))
-  (segment (start 52.07 41.91) (end 59.055 41.91) (width 0.5) (layer B.Cu) (net 10))
-  (segment (start 22.86 30.48) (end 25.4 30.48) (width 0.5) (layer B.Cu) (net 10))
-  (segment (start 25.4 41.91) (end 25.4 30.48) (width 0.5) (layer B.Cu) (net 10))
-  (segment (start 25.4 30.48) (end 25.4 27.94) (width 0.5) (layer B.Cu) (net 10))
-  (segment (start 49.53 25.4) (end 49.53 31.75) (width 0.5) (layer B.Cu) (net 10))
-  (segment (start 49.53 31.75) (end 49.53 36.83) (width 0.5) (layer B.Cu) (net 10))
-  (segment (start 27.94 25.4) (end 49.53 25.4) (width 0.5) (layer B.Cu) (net 10))
-  (segment (start 25.4 27.94) (end 27.94 25.4) (width 0.5) (layer B.Cu) (net 10))
-  (segment (start 49.53 36.83) (end 49.53 39.37) (width 0.5) (layer B.Cu) (net 10))
-  (segment (start 22.86 41.91) (end 25.4 41.91) (width 0.5) (layer B.Cu) (net 10))
+  (segment (start 44.45 43.815) (end 48.26 43.815) (width 0.75) (layer B.Cu) (net 8))
+  (segment (start 48.26 41.275) (end 47.625 41.275) (width 0.75) (layer B.Cu) (net 10))
+  (segment (start 47.625 41.275) (end 45.085 38.735) (width 0.75) (layer B.Cu) (net 10))
+  (segment (start 45.085 38.735) (end 44.45 38.735) (width 0.75) (layer B.Cu) (net 10))
+  (segment (start 25.4 53.34) (end 25.4 62.23) (width 0.75) (layer B.Cu) (net 10))
+  (segment (start 25.4 62.23) (end 22.86 64.77) (width 0.75) (layer B.Cu) (net 10))
+  (segment (start 25.4 41.91) (end 25.4 53.34) (width 0.75) (layer B.Cu) (net 10))
+  (segment (start 25.4 53.34) (end 22.86 53.34) (width 0.75) (layer B.Cu) (net 10))
+  (segment (start 22.86 30.48) (end 25.4 30.48) (width 0.75) (layer B.Cu) (net 10))
+  (segment (start 25.4 41.91) (end 25.4 30.48) (width 0.75) (layer B.Cu) (net 10))
+  (segment (start 25.4 30.48) (end 25.4 27.94) (width 0.75) (layer B.Cu) (net 10))
+  (segment (start 44.45 25.4) (end 44.45 31.75) (width 0.75) (layer B.Cu) (net 10))
+  (segment (start 44.45 31.75) (end 44.45 34.29) (width 0.75) (layer B.Cu) (net 10) (status 20))
+  (segment (start 44.45 34.29) (end 44.45 36.195) (width 0.75) (layer B.Cu) (net 10) (status 20))
+  (segment (start 27.94 25.4) (end 44.45 25.4) (width 0.75) (layer B.Cu) (net 10))
+  (segment (start 25.4 27.94) (end 27.94 25.4) (width 0.75) (layer B.Cu) (net 10))
+  (segment (start 44.45 36.195) (end 44.45 38.735) (width 0.75) (layer B.Cu) (net 10) (status 30))
+  (segment (start 22.86 41.91) (end 25.4 41.91) (width 0.75) (layer B.Cu) (net 10))
+  (segment (start 44.45 41.275) (end 45.085 41.275) (width 0.75) (layer B.Cu) (net 14))
+  (segment (start 47.625 38.735) (end 48.26 38.735) (width 0.75) (layer B.Cu) (net 14))
   (segment (start 22.86 36.91) (end 22.94 36.83) (width 0.25) (layer F.Cu) (net 14))
   (zone (net 14) (net_name "Net-(J1-Pad6)") (layer B.Cu) (hatch edge 0.508)
-    (connect_pads (clearance 0.508))
-    (min_thickness 0.254)
-    (fill yes (arc_segments 16) (thermal_gap 0.508) (thermal_bridge_width 0.508))
+    (connect_pads (clearance 0.8))
+    (min_thickness 0.7)
+    (fill yes (arc_segments 16) (thermal_gap 0.8) (thermal_bridge_width 0.8))
     (polygon
       (pts
-        (xy 71.12 69.85) (xy 19.685 69.85) (xy 19.685 20.955) (xy 71.12 20.955)
+        (xy 56.515 67.945) (xy 19.685 67.945) (xy 19.685 22.225) (xy 56.515 22.225)
       )
     )
