File: Platinen/Taster/taster.kicad_pcb (KiCad board)
At the start: 2 copper layers, 4 parts, among them J1 CONN_01X03_FEMALE, SW1 SW_Push

Commit message: Platinen aktuallisiert nach Ätzen der ersten Prototypplatine
Routing:
- net Net-(R1-Pad2): track 19.9 -> 21.2 mm
Changed lines of the file:
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@@
-(kicad_pcb (version 4) (host pcbnew 4.0.6-e0-6349~53~ubuntu14.04.1)
+(kicad_pcb (version 4) (host pcbnew 4.0.7-e2-6376~58~ubuntu16.04.1)
   (general
     (links 7)
     (no_connects 2)
-    (area 147.32 102.045 190.500001 113.955)
+    (area 147.32 101.6 190.500001 113.955)
     (thickness 1.6)
-    (drawings 0)
+    (drawings 1)
     (tracks 13)
     (zones 0)
@@
     )
   )
+  (dimension 10.16 (width 0.3) (layer F.Adhes)
+    (gr_text "10,160 mm" (at 182.88 96.44) (layer F.Adhes)
+      (effects (font (size 1.5 1.5) (thickness 0.3)))
+    )
+    (feature1 (pts (xy 187.96 100.33) (xy 187.96 95.09)))
+    (feature2 (pts (xy 177.8 100.33) (xy 177.8 95.09)))
+    (crossbar (pts (xy 177.8 97.79) (xy 187.96 97.79)))
+    (arrow1a (pts (xy 187.96 97.79) (xy 186.833496 98.376421)))
+    (arrow1b (pts (xy 187.96 97.79) (xy 186.833496 97.203579)))
+    (arrow2a (pts (xy 177.8 97.79) (xy 178.926504 98.376421)))
+    (arrow2b (pts (xy 177.8 97.79) (xy 178.926504 97.203579)))
+  )
   (segment (start 172.72 105.41) (end 176.53 105.41) (width 0.4) (layer B.Cu) (net 1))
   (segment (start 176.53 107.95) (end 160.02 107.95) (width 0.4) (layer B.Cu) (net 2))
@@
   (segment (start 154.94 107.95) (end 157.48 110.49) (width 0.4) (layer B.Cu) (net 4))
   (segment (start 154.94 105.41) (end 154.94 107.95) (width 0.4) (layer B.Cu) (net 4))
-  (segment (start 156.21 104.14) (end 154.94 105.41) (width 0.4) (layer B.Cu) (net 4))
-  (segment (start 158.75 104.14) (end 156.21 104.14) (width 0.4) (layer B.Cu) (net 4))
-  (segment (start 160.02 105.41) (end 158.75 104.14) (width 0.4) (layer B.Cu) (net 4))
+  (segment (start 155.575 103.505) (end 154.94 105.41) (width 0.4) (layer B.Cu) (net 4))
+  (segment (start 158.75 103.505) (end 155.575 103.505) (width 0.4) (layer B.Cu) (net 4))
+  (segment (start 160.02 105.41) (end 158.75 103.505) (width 0.4) (layer B.Cu) (net 4))
   (segment (start 162.56 105.41) (end 160.02 105.41) (width 0.4) (layer B.Cu) (net 4))
   (segment (start 157.48 110.49) (end 162.56 110.49) (width 0.4) (layer B.Cu) (net 4))
@@
     (polygon
       (pts
-        (xy 147.32 102.87) (xy 147.32 113.03) (xy 190.5 113.03) (xy 190.5 102.87)
+        (xy 147.32 101.6) (xy 147.32 113.03) (xy 187.96 113.03) (xy 187.96 101.6)
       )
     )

Commit message: Platinen überarbeitet
Parts:
- moved SW1 1.27 mm to (158.8, 110.5)
Routing:
- net Net-(R1-Pad2): track 21.2 -> 18.2 mm
Other:
- net class Default: trace_width 0.4 -> 0.75
- board text added: "3,3V"
- board text added: "GND"
- board text added: "PIN"
Changed lines of the file:
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@@
     (links 7)
     (no_connects 2)
-    (area 147.32 101.6 190.500001 113.955)
+    (area 149.86 102.045 185.420001 113.955)
     (thickness 1.6)
-    (drawings 1)
-    (tracks 13)
+    (drawings 3)
+    (tracks 14)
     (zones 0)
     (modules 4)
@@
   )
   (setup
-    (last_trace_width 0.4)
+    (last_trace_width 0.75)
     (trace_clearance 0.2)
-    (zone_clearance 0.508)
+    (zone_clearance 0.8)
     (zone_45_only no)
     (trace_min 0.2)
@@
     (pad_drill 1)
     (pad_to_mask_clearance 0.2)
-    (aux_axis_origin 0 0)
+    (aux_axis_origin 149.86 113.03)
+    (grid_origin 149.86 113.03)
     (visible_elements FFFFFF7F)
     (pcbplotparams
-      (layerselection 0x00030_80000001)
+      (layerselection 0x00008_80000000)
       (usegerberextensions false)
       (excludeedgelayer true)
@@
       (viasonmask false)
       (mode 1)
-      (useauxorigin false)
+      (useauxorigin true)
       (hpglpennumber 1)
       (hpglpenspeed 20)
@@
       (psnegative false)
       (psa4output false)
-      (plotreference true)
-      (plotvalue true)
+      (plotreference false)
+      (plotvalue false)
       (plotinvisibletext false)
       (padsonsilk false)
@@
       (outputformat 1)
       (mirror false)
-      (drillshape 1)
+      (drillshape 0)
       (scaleselection 1)
       (outputdirectory ""))
@@
   (net_class Default "Dies ist die voreingestellte Netzklasse."
     (clearance 0.2)
-    (trace_width 0.4)
+    (trace_width 0.75)
     (via_dia 0.6)
     (via_drill 0.4)
@@
   )
   (module Buttons_Switches_THT:SW_PUSH_6mm (layer F.Cu)
-    (at 157.48 110.49 180)
+    (at 158.75 110.49 180)
     (descr https://www.omron.com/ecb/products/pdf/en-b3f.pdf)
     (tags "tact sw push 6mm")
@@
     )
   )
-  (dimension 10.16 (width 0.3) (layer F.Adhes)
-    (gr_text "10,160 mm" (at 182.88 96.44) (layer F.Adhes)
-      (effects (font (size 1.5 1.5) (thickness 0.3)))
-    )
-    (feature1 (pts (xy 187.96 100.33) (xy 187.96 95.09)))
-    (feature2 (pts (xy 177.8 100.33) (xy 177.8 95.09)))
-    (crossbar (pts (xy 177.8 97.79) (xy 187.96 97.79)))
-    (arrow1a (pts (xy 187.96 97.79) (xy 186.833496 98.376421)))
-    (arrow1b (pts (xy 187.96 97.79) (xy 186.833496 97.203579)))
-    (arrow2a (pts (xy 177.8 97.79) (xy 178.926504 98.376421)))
-    (arrow2b (pts (xy 177.8 97.79) (xy 178.926504 97.203579)))
-  )
-  (segment (start 172.72 105.41) (end 176.53 105.41) (width 0.4) (layer B.Cu) (net 1))
-  (segment (start 176.53 107.95) (end 160.02 107.95) (width 0.4) (layer B.Cu) (net 2))
-  (segment (start 160.02 107.95) (end 158.06 105.99) (width 0.4) (layer B.Cu) (net 2))
-  (segment (start 158.06 105.99) (end 157.48 105.99) (width 0.4) (layer B.Cu) (net 2))
-  (segment (start 157.48 105.99) (end 158.06 105.99) (width 0.25) (layer B.Cu) (net 2))
-  (segment (start 176.53 110.49) (end 172.72 110.49) (width 0.4) (layer B.Cu) (net 3))
-  (segment (start 154.94 107.95) (end 157.48 110.49) (width 0.4) (layer B.Cu) (net 4))
-  (segment (start 154.94 105.41) (end 154.94 107.95) (width 0.4) (layer B.Cu) (net 4))
-  (segment (start 155.575 103.505) (end 154.94 105.41) (width 0.4) (layer B.Cu) (net 4))
-  (segment (start 158.75 103.505) (end 155.575 103.505) (width 0.4) (layer B.Cu) (net 4))
-  (segment (start 160.02 105.41) (end 158.75 103.505) (width 0.4) (layer B.Cu) (net 4))
-  (segment (start 162.56 105.41) (end 160.02 105.41) (width 0.4) (layer B.Cu) (net 4))
-  (segment (start 157.48 110.49) (end 162.56 110.49) (width 0.4) (layer B.Cu) (net 4))
+  (gr_text 3,3V (at 179.07 107.95) (layer F.Paste)
+    (effects (font (size 1.8 1.8) (thickness 0.1)) (justify left))
+  )
+  (gr_text PIN (at 179.07 105.41) (layer F.Paste)
+    (effects (font (size 1.8 1.8) (thickness 0.1)) (justify left))
+  )
+  (gr_text GND (at 179.07 110.49) (layer F.Paste)
+    (effects (font (size 1.8 1.8) (thickness 0.1)) (justify left))
+  )
+  (segment (start 172.72 105.41) (end 176.53 105.41) (width 0.75) (layer B.Cu) (net 1))
+  (segment (start 158.75 105.99) (end 158.75 106.68) (width 0.75) (layer B.Cu) (net 2))
+  (segment (start 158.75 106.68) (end 160.02 107.95) (width 0.75) (layer B.Cu) (net 2))
+  (segment (start 160.02 107.95) (end 176.53 107.95) (width 0.75) (layer B.Cu) (net 2))
+  (segment (start 159.33 105.99) (end 158.75 105.99) (width 0.4) (layer B.Cu) (net 2) (status 30))
+  (segment (start 158.75 105.99) (end 159.33 105.99) (width 0.25) (layer B.Cu) (net 2) (status 30))
+  (segment (start 176.53 110.49) (end 172.72 110.49) (width 0.75) (layer B.Cu) (net 3))
+  (segment (start 162.56 105.41) (end 161.925 105.41) (width 0.75) (layer B.Cu) (net 4))
+  (segment (start 161.925 105.41) (end 160.02 103.505) (width 0.75) (layer B.Cu) (net 4))
+  (segment (start 160.02 103.505) (end 157.48 103.505) (width 0.75) (layer B.Cu) (net 4))
+  (segment (start 157.48 103.505) (end 156.21 104.775) (width 0.75) (layer B.Cu) (net 4))
+  (segment (start 156.21 104.775) (end 156.21 107.95) (width 0.75) (layer B.Cu) (net 4))
+  (segment (start 156.21 107.95) (end 158.75 110.49) (width 0.75) (layer B.Cu) (net 4))
+  (segment (start 158.75 110.49) (end 162.56 110.49) (width 0.75) (layer B.Cu) (net 4) (status 10))
   (zone (net 3) (net_name "Net-(J1-Pad3)") (layer B.Cu) (hatch edge 0.508)
-    (connect_pads (clearance 0.508))
-    (min_thickness 0.254)
-    (fill yes (arc_segments 16) (thermal_gap 0.508) (thermal_bridge_width 0.508))
+    (connect_pads (clearance 0.8))
+    (min_thickness 0.7)
+    (fill yes (arc_segments 16) (thermal_gap 0.8) (thermal_bridge_width 0.8))
     (polygon
       (pts
-        (xy 147.32 101.6) (xy 147.32 113.03) (xy 187.96 113.03) (xy 187.96 101.6)
+        (xy 149.86 102.87) (xy 149.86 113.03) (xy 185.42 113.03) (xy 185.42 102.87)
       )
     )
